Commit message: Add Gazebo control and launch files for robot simulation

File: src/articubot_one/description/robot_core.xacro (robot description, xacro)
@@ -59,4 +59,7 @@
       </xacro:inertial_box>
     </link>
+    <gazebo reference="chassis">
+      <material>Gazebo/White</material>
+    </gazebo>
     <joint name="left_wheel_joint" type="continuous">
       <parent link="chassis"/>
@@ -81,4 +84,7 @@
     </xacro:inertial_cylinder>
     </link>
+    <gazebo reference="left_wheel">
+      <material>Gazebo/Orange</material>
+    </gazebo>
     <joint name="right_wheel_joint" type="continuous">
       <parent link="chassis"/>
@@ -103,4 +109,7 @@
     </xacro:inertial_cylinder>
     </link>
+    <gazebo reference="right_wheel">
+      <material>Gazebo/Orange</material>
+    </gazebo>
     <joint name="caster_wheel_joint" type="fixed">
      <parent link="chassis"/>
@@ -126,3 +135,6 @@
       </xacro:inertial_sphere>
     </link>
+    <gazebo reference="caster_wheel">
+      <material>Gazebo/Red</material>
+    </gazebo>
 </robot>
